File: ct_input.sch (KiCad schematic (older format))
At the start: 2 parts, among them J11 AudioJack3

Commit message: little modifications
Changed lines of the file:
@@
 $Descr A4 11693 8268
 encoding utf-8
-Sheet 8 15
+Sheet 3 15
 Title ""
 Date ""
@@
 AR Path="/61074E24/6115FA69/610A585F" Ref="R19"  Part="1"
 AR Path="/61150CE0/6115FA69/610A585F" Ref="R13"  Part="1"
-F 0 "R19" H 2070 1096 50  0000 L CNN
+F 0 "R8" H 2070 1096 50  0000 L CNN
 F 1 "100" H 2070 1005 50  0000 L CNN
 F 2 "Resistor_SMD:R_0805_2012Metric" V 1930 1050 50  0001 C CNN
@@
 AR Path="/61074E24/610A9775/6116D55F" Ref="J15"  Part="1"
 AR Path="/61074E24/6115FA69/6116D55F" Ref="J16"  Part="1"
-F 0 "J16" H 1182 1375 50  0000 C CNN
+F 0 "J5" H 1182 1375 50  0000 C CNN
 F 1 "AudioJack3" H 1182 1284 50  0000 C CNN
 F 2 "project_lib:C18594" H 1200 1050 50  0001 C CNN
