File: esp32_energy_meter.kicad_pcb (KiCad board)
At the start: 2 copper layers, 90 x 100 mm, 75 parts, among them IC1 REF2933AIDBZR, IC2 ADC128S102CIMTX_NOPB, IC3 ADC128S102CIMTX_NOPB, J1 Screw_Terminal_01x02, J10 AudioJack3, J11 AudioJack3, J12 AudioJack3, J13 AudioJack3, J14 AudioJack3, J15 AudioJack3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

Commit message: little modifications
Changed lines of the file:
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@@
     (solder_mask_min_width 0.25)
     (aux_axis_origin 0 0)
-    (visible_elements FFFFFF7F)
+    (visible_elements 7FFFFFFF)
     (pcbplotparams
       (layerselection 0x010fc_ffffffff)
@@
   (via (at 169.418 73.914) (size 0.8) (drill 0.4) (layers F.Cu B.Cu) (net 16))
   (via (at 173.228 77.978) (size 0.8) (drill 0.4) (layers F.Cu B.Cu) (net 16))
-  (via (at 179.07 70.612) (size 0.8) (drill 0.4) (layers F.Cu B.Cu) (net 16))
+  (via (at 177.038 73.152) (size 0.8) (drill 0.4) (layers F.Cu B.Cu) (net 16))
   (via (at 156.464 73.152) (size 0.8) (drill 0.4) (layers F.Cu B.Cu) (net 16))
   (via (at 156.464 78.232) (size 0.8) (drill 0.4) (layers F.Cu B.Cu) (net 16))
@@
   (via (at 151.13 55.88) (size 0.8) (drill 0.4) (layers F.Cu B.Cu) (net 16))
   (via (at 151.384 66.802) (size 0.8) (drill 0.4) (layers F.Cu B.Cu) (net 16))
+  (segment (start 174.371 69.244) (end 172.691 67.564) (width 0.25) (layer F.Cu) (net 17))
+  (segment (start 174.371 70.494) (end 174.371 69.244) (width 0.25) (layer F.Cu) (net 17))
+  (segment (start 169.833 66.486) (end 169.833 65.786) (width 0.25) (layer F.Cu) (net 17))
+  (segment (start 170.911 67.564) (end 169.833 66.486) (width 0.25) (layer F.Cu) (net 17))
+  (segment (start 172.691 67.564) (end 170.911 67.564) (width 0.25) (layer F.Cu) (net 17))
+  (segment (start 169.65 62.1295) (end 169.7505 62.23) (width 0.25) (layer F.Cu) (net 17))
+  (segment (start 169.65 58.07) (end 169.65 62.1295) (width 0.25) (layer F.Cu) (net 17))
+  (segment (start 169.7505 65.7035) (end 169.833 65.786) (width 0.25) (layer F.Cu) (net 17))
+  (segment (start 169.7505 62.23) (end 169.7505 65.7035) (width 0.25) (layer F.Cu) (net 17))
   (segment (start 134.80138 122.865) (end 135.50138 122.165) (width 0.25) (layer F.Cu) (net 18))
   (segment (start 131.17498 122.865) (end 134.80138 122.865) (width 0.25) (layer F.Cu) (net 18))
@@
   (segment (start 153.924 109.541919) (end 157.279839 106.18608) (width 0.25) (layer F.Cu) (net 18))
   (segment (start 153.924 110.744) (end 153.924 109.541919) (width 0.25) (layer F.Cu) (net 18))
-  (segment (start 175.0949 145.034) (end 176.32426 146.26336) (width 0.5) (layer F.Cu) (net 71))
-  (segment (start 164.338 145.034) (end 175.0949 145.034) (width 0.5) (layer F.Cu) (net 71))
-  (segment (start 164.338 147.15532) (end 162.90332 148.59) (width 0.5) (layer F.Cu) (net 71))
-  (segment (start 164.338 145.034) (end 164.338 147.15532) (width 0.5) (layer F.Cu) (net 71))
-  (segment (start 154.41998 148.59) (end 153.12644 147.29646) (width 0.5) (layer F.Cu) (net 71))
-  (segment (start 162.90332 148.59) (end 154.41998 148.59) (width 0.5) (layer F.Cu) (net 71))
-  (segment (start 159.258 143.034) (end 160.56 141.732) (width 0.5) (layer F.Cu) (net 72))
-  (segment (start 159.258 145.034) (end 159.258 143.034) (width 0.5) (layer F.Cu) (net 72))
-  (segment (start 176.7929 141.732) (end 181.32426 146.26336) (width 0.5) (layer F.Cu) (net 72))
-  (segment (start 165.38194 136.87806) (end 160.528 141.732) (width 0.5) (layer F.Cu) (net 72))
-  (segment (start 160.56 141.732) (end 160.528 141.732) (width 0.5) (layer F.Cu) (net 72))
-  (segment (start 165.38194 135.51662) (end 165.38194 136.87806) (width 0.5) (layer F.Cu) (net 72))
-  (segment (start 160.528 141.732) (end 176.7929 141.732) (width 0.5) (layer F.Cu) (net 72))
   (segment (start 130.24768 96.824) (end 130.19768 96.774) (width 0.25) (layer F.Cu) (net 19))
   (segment (start 167.70056 109.21566) (end 167.70056 108.6498) (width 0.5) (layer F.Cu) (net 19))
@@
   (segment (start 153.12644 135.96112) (end 152.68194 135.51662) (width 0.5) (layer F.Cu) (net 48))
   (segment (start 153.12644 141.49646) (end 153.12644 135.96112) (width 0.5) (layer F.Cu) (net 48))
-  (segment (start 174.371 69.244) (end 172.691 67.564) (width 0.25) (layer F.Cu) (net 17))
-  (segment (start 174.371 70.494) (end 174.371 69.244) (width 0.25) (layer F.Cu) (net 17))
-  (segment (start 169.833 66.486) (end 169.833 65.786) (width 0.25) (layer F.Cu) (net 17))
-  (segment (start 170.911 67.564) (end 169.833 66.486) (width 0.25) (layer F.Cu) (net 17))
-  (segment (start 172.691 67.564) (end 170.911 67.564) (width 0.25) (layer F.Cu) (net 17))
-  (segment (start 169.65 62.1295) (end 169.7505 62.23) (width 0.25) (layer F.Cu) (net 17))
-  (segment (start 169.65 58.07) (end 169.65 62.1295) (width 0.25) (layer F.Cu) (net 17))
-  (segment (start 169.7505 65.7035) (end 169.833 65.786) (width 0.25) (layer F.Cu) (net 17))
-  (segment (start 169.7505 62.23) (end 169.7505 65.7035) (width 0.25) (layer F.Cu) (net 17))
   (segment (start 131.17498 120.44) (end 131.17498 120.915) (width 0.25) (layer F.Cu) (net 49))
   (segment (start 157.48 94.996) (end 132.036 120.44) (width 0.25) (layer F.Cu) (net 49))
@@
   (segment (start 158.942 58.8495) (end 158.242 58.8495) (width 0.25) (layer F.Cu) (net 70))
   (segment (start 170.561 70.494) (end 170.561 69.244) (width 0.25) (layer F.Cu) (net 70))
+  (segment (start 175.0949 145.034) (end 176.32426 146.26336) (width 0.5) (layer F.Cu) (net 71))
+  (segment (start 164.338 145.034) (end 175.0949 145.034) (width 0.5) (layer F.Cu) (net 71))
+  (segment (start 164.338 147.15532) (end 162.90332 148.59) (width 0.5) (layer F.Cu) (net 71))
+  (segment (start 164.338 145.034) (end 164.338 147.15532) (width 0.5) (layer F.Cu) (net 71))
+  (segment (start 154.41998 148.59) (end 153.12644 147.29646) (width 0.5) (layer F.Cu) (net 71))
+  (segment (start 162.90332 148.59) (end 154.41998 148.59) (width 0.5) (layer F.Cu) (net 71))
+  (segment (start 159.258 143.034) (end 160.56 141.732) (width 0.5) (layer F.Cu) (net 72))
+  (segment (start 159.258 145.034) (end 159.258 143.034) (width 0.5) (layer F.Cu) (net 72))
+  (segment (start 176.7929 141.732) (end 181.32426 146.26336) (width 0.5) (layer F.Cu) (net 72))
+  (segment (start 165.38194 136.87806) (end 160.528 141.732) (width 0.5) (layer F.Cu) (net 72))
+  (segment (start 160.56 141.732) (end 160.528 141.732) (width 0.5) (layer F.Cu) (net 72))
+  (segment (start 165.38194 135.51662) (end 165.38194 136.87806) (width 0.5) (layer F.Cu) (net 72))
+  (segment (start 160.528 141.732) (end 176.7929 141.732) (width 0.5) (layer F.Cu) (net 72))
   (zone (net 16) (net_name GND) (layer F.Cu) (hatch edge 0.508)
     (connect_pads (clearance 0.25))
@@
     (polygon
       (pts
-        (xy 190.754 49.52238) (xy 190.5 128.016) (xy 167.64 128.016) (xy 167.64 115.316) (xy 141.224 115.316)
-        (xy 141.224 49.657)
+        (xy 190.754 49.52238) (xy 190.754 64.516) (xy 178.308 64.516) (xy 178.308 93.218) (xy 190.246 93.218)
+        (xy 190.5 128.016) (xy 167.64 128.016) (xy 167.64 115.316) (xy 141.224 115.316) (xy 141.224 49.657)
       )
     )
@@
     (polygon
       (pts
-        (xy 190.754 49.52238) (xy 190.5 128.016) (xy 167.64 128.016) (xy 167.64 115.316) (xy 141.224 115.316)
-        (xy 141.224 49.657)
+        (xy 190.754 49.52238) (xy 190.754 64.516) (xy 178.308 64.516) (xy 178.308 93.218) (xy 190.246 93.218)
+        (xy 190.5 128.016) (xy 167.64 128.016) (xy 167.64 115.316) (xy 141.224 115.316) (xy 141.224 49.657)
       )
     )
