File: esp32_energy_meter.sch (KiCad schematic (older format))
At the start: 41 parts, among them IC1 REF2933AIDBZR, J1 Screw_Terminal_01x02, J2 Conn_01x06_MountingPin, J3 Conn_02x02_Top_Bottom, J4 Conn_01x06_MountingPin, SW1 SW_Push, SW2 SW_Push, U1 ESP32-WROOM-32, U2 LM1117-3.3

Commit message: little modifications
Parts:
- TP1, TP2, TP3, TP4, TP5, TP6, TP7, TP8: LCSC (none) -> x
Changed lines of the file:
@@
 F4 "DOUT" I L 7750 1200 50
 F5 "DIN" I L 7750 1100 50
-F7 "IN6" O R 8450 1250 50
-F8 "IN7" O R 8450 1400 50
+F6 "IN6" O R 8450 1250 50
+F7 "IN7" O R 8450 1400 50
 $EndSheet
 Wire Wire Line
@@
 F 2 "TestPoint:TestPoint_Pad_1.0x1.0mm" H 9500 2000 50  0001 C CNN
 F 3 "~" H 9500 2000 50  0001 C CNN
+F 4 "x" H 9300 2000 50  0001 C CNN "LCSC"
 	1    9300 2000
 	0    1    1    0
@@
 F 2 "TestPoint:TestPoint_Pad_1.0x1.0mm" H 9500 1850 50  0001 C CNN
 F 3 "~" H 9500 1850 50  0001 C CNN
+F 4 "x" H 9300 1850 50  0001 C CNN "LCSC"
 	1    9300 1850
 	0    1    1    0
@@
 F 2 "TestPoint:TestPoint_Pad_1.0x1.0mm" H 9500 1750 50  0001 C CNN
 F 3 "~" H 9500 1750 50  0001 C CNN
+F 4 "x" H 9300 1750 50  0001 C CNN "LCSC"
 	1    9300 1750
 	0    1    1    0
@@
 F 2 "TestPoint:TestPoint_Pad_1.0x1.0mm" H 9500 1650 50  0001 C CNN
 F 3 "~" H 9500 1650 50  0001 C CNN
+F 4 "x" H 9300 1650 50  0001 C CNN "LCSC"
 	1    9300 1650
 	0    1    1    0
@@
 F 2 "TestPoint:TestPoint_Pad_1.0x1.0mm" H 9500 2850 50  0001 C CNN
 F 3 "~" H 9500 2850 50  0001 C CNN
+F 4 "x" H 9300 2850 50  0001 C CNN "LCSC"
 	1    9300 2850
 	0    1    1    0
@@
 F 2 "TestPoint:TestPoint_Pad_1.0x1.0mm" H 9500 2700 50  0001 C CNN
 F 3 "~" H 9500 2700 50  0001 C CNN
+F 4 "x" H 9300 2700 50  0001 C CNN "LCSC"
 	1    9300 2700
 	0    1    1    0
@@
 F 2 "TestPoint:TestPoint_Pad_1.0x1.0mm" H 9500 2600 50  0001 C CNN
 F 3 "~" H 9500 2600 50  0001 C CNN
+F 4 "x" H 9300 2600 50  0001 C CNN "LCSC"
 	1    9300 2600
 	0    1    1    0
@@
 F 2 "TestPoint:TestPoint_Pad_1.0x1.0mm" H 9500 2500 50  0001 C CNN
 F 3 "~" H 9500 2500 50  0001 C CNN
+F 4 "x" H 9300 2500 50  0001 C CNN "LCSC"
 	1    9300 2500
 	0    1    1    0
