File: measurement.sch (KiCad schematic (older format))
At the start: 4 parts, among them IC3 ADC128S102CIMTX_NOPB

Commit message: little modifications
Changed lines of the file:
@@
 $Descr A4 11693 8268
 encoding utf-8
-Sheet 9 15
+Sheet 2 15
 Title ""
 Date ""
@@
 AR Path="/61149304/61077634" Ref="#PWR?"  Part="1"
 AR Path="/61150CE0/61077634" Ref="#PWR035"  Part="1"
-F 0 "#PWR044" H 3100 2100 50  0001 C CNN
+F 0 "#PWR035" H 3100 2100 50  0001 C CNN
 F 1 "GNDA" H 3105 2177 50  0000 C CNN
 F 2 "" H 3100 2350 50  0001 C CNN
@@
 AR Path="/61149304/6107763B" Ref="#PWR?"  Part="1"
 AR Path="/61150CE0/6107763B" Ref="#PWR037"  Part="1"
-F 0 "#PWR046" H 4750 2300 50  0001 C CNN
+F 0 "#PWR037" H 4750 2300 50  0001 C CNN
 F 1 "GND" H 4755 2377 50  0000 C CNN
 F 2 "" H 4750 2550 50  0001 C CNN
@@
 AR Path="/61149304/61077642" Ref="#PWR?"  Part="1"
 AR Path="/61150CE0/61077642" Ref="#PWR036"  Part="1"
-F 0 "#PWR045" H 4900 2250 50  0001 C CNN
+F 0 "#PWR036" H 4900 2250 50  0001 C CNN
 F 1 "+3.3V" H 4915 2573 50  0000 C CNN
 F 2 "" H 4900 2400 50  0001 C CNN
@@
 AR Path="/61149304/610B2F25" Ref="C?"  Part="1"
 AR Path="/61150CE0/610B2F25" Ref="C11"  Part="1"
-F 0 "C14" H 4015 1046 50  0000 L CNN
+F 0 "C11" H 4015 1046 50  0000 L CNN
 F 1 "1uf" H 4015 955 50  0000 L CNN
 F 2 "Capacitor_SMD:C_0805_2012Metric_Pad1.15x1.40mm_HandSolder" H 3938 850 50  0001 C CNN
@@
 AR Path="/61149304/610B4066" Ref="#PWR?"  Part="1"
 AR Path="/61150CE0/610B4066" Ref="#PWR030"  Part="1"
-F 0 "#PWR039" H 3900 650 50  0001 C CNN
+F 0 "#PWR030" H 3900 650 50  0001 C CNN
 F 1 "+3.3V" H 3915 973 50  0000 C CNN
 F 2 "" H 3900 800 50  0001 C CNN
@@
 AR Path="/61149304/610B48E9" Ref="#PWR?"  Part="1"
 AR Path="/61150CE0/610B48E9" Ref="#PWR032"  Part="1"
-F 0 "#PWR041" H 3900 950 50  0001 C CNN
+F 0 "#PWR032" H 3900 950 50  0001 C CNN
 F 1 "GND" H 3905 1027 50  0000 C CNN
 F 2 "" H 3900 1200 50  0001 C CNN
@@
 AR Path="/61149304/6107762E" Ref="IC?"  Part="1"
 AR Path="/61150CE0/6107762E" Ref="IC2"  Part="1"
-F 0 "IC3" H 3950 2415 50  0000 C CNN
+F 0 "IC2" H 3950 2415 50  0000 C CNN
 F 1 "ADC128S102CIMTX_NOPB" H 3950 2324 50  0000 C CNN
 F 2 "SOP65P640X120-16N" H 4350 2250 50  0001 L CNN
@@
 AR Path="/61149304/610BB1B8" Ref="#PWR?"  Part="1"
 AR Path="/61150CE0/610BB1B8" Ref="#PWR033"  Part="1"
-F 0 "#PWR042" H 4550 950 50  0001 C CNN
+F 0 "#PWR033" H 4550 950 50  0001 C CNN
 F 1 "GNDA" H 4555 1027 50  0000 C CNN
 F 2 "" H 4550 1200 50  0001 C CNN
@@
 AR Path="/61149304/610B8D10" Ref="C?"  Part="1"
 AR Path="/61150CE0/610B8D10" Ref="C9"  Part="1"
-F 0 "C12" H 4665 996 50  0000 L CNN
+F 0 "C9" H 4665 996 50  0000 L CNN
 F 1 "100nf" H 4665 905 50  0000 L CNN
 F 2 "Capacitor_SMD:C_0805_2012Metric_Pad1.15x1.40mm_HandSolder" H 4588 800 50  0001 C CNN
@@
 AR Path="/61149304/610B04E2" Ref="C?"  Part="1"
 AR Path="/61150CE0/610B04E2" Ref="C10"  Part="1"
-F 0 "C13" H 3265 1046 50  0000 L CNN
+F 0 "C10" H 3265 1046 50  0000 L CNN
 F 1 "100nf" H 3265 955 50  0000 L CNN
 F 2 "Capacitor_SMD:C_0805_2012Metric_Pad1.15x1.40mm_HandSolder" H 3188 850 50  0001 C CNN
@@
 AR Path="/61149304/610F54A9" Ref="#PWR?"  Part="1"
 AR Path="/61150CE0/610F54A9" Ref="#PWR034"  Part="1"
-F 0 "#PWR043" H 3050 2050 50  0001 C CNN
+F 0 "#PWR034" H 3050 2050 50  0001 C CNN
 F 1 "+3.3VA" H 3065 2373 50  0000 C CNN
 F 2 "" H 3050 2200 50  0001 C CNN
@@
 AR Path="/61149304/610FB67B" Ref="#PWR?"  Part="1"
 AR Path="/61150CE0/610FB67B" Ref="#PWR029"  Part="1"
-F 0 "#PWR038" H 3150 650 50  0001 C CNN
+F 0 "#PWR029" H 3150 650 50  0001 C CNN
 F 1 "+3.3VA" H 3165 973 50  0000 C CNN
 F 2 "" H 3150 800 50  0001 C CNN
@@
 AR Path="/61149304/610FC15E" Ref="#PWR?"  Part="1"
 AR Path="/61150CE0/610FC15E" Ref="#PWR031"  Part="1"
-F 0 "#PWR040" H 3150 900 50  0001 C CNN
+F 0 "#PWR031" H 3150 900 50  0001 C CNN
 F 1 "GNDA" H 3155 977 50  0000 C CNN
 F 2 "" H 3150 1150 50  0001 C CNN
